File: Episode 24 Pyramiduino PCB/Exercise/Pyramiduino-two final nets.kicad_pcb (KiCad board)
At the start: 2 copper layers, 52.6 x 45.6 mm, 23 parts, among them IC1 ATMEGA328-A, P1 CONN_01X16, P2 CONN_01X14, P3 CONN_01X14, P4 CONN_01X01, P5 CONN_01X01, P6 CONN_01X01, SW1 SW_PUSH, U1 MIC5504-3.3YM5, Y1 16M

Commit message: Correction of reset, MOSI and MISO nets.
Given the Piramiduino-two schematics some changes were made in order order to correct and improve the PCB project. Also some Vias were deleted and other connections made.
Other:
- net class Default removed
- net class Power removed
